File: peaks/hardware_design/pcb_banana/peaks_v02.sch (EAGLE design)
At the start: 92 parts, among them IC1 LM1117-3.3, IC2 LM4040B25, IC3 DAC8552, IC4 OPA2171, IC5 OPA2171, IC6 LM4040B10, Q1 8MHz, Q2 MMBT3904, Q3 MMBT3904, SW3 EVQQ2, SW5 EVQQ2

Commit message: adding rapid bananas
Parts:
- removed TRIG1IN, TRIG2IN: (no value), Jalco_3_5_jack:YKB21-5129
- added TRIG1, TRIG2: WQP-PJ301BM, minijack_3_5_quingpu:WQP-PJ301BM
- OUTA, OUTB: value (none) -> WQP-PJ301BM; device Jalco_3_5_jack:YKB21-5129 -> minijack_3_5_quingpu:WQP-PJ301BM
- renumbered SWTRIG1 to SW6, SWTRIG2 to SW4
Connections:
- net GND: now also TRIG1.SLEVE, TRIG1.SWITCH, TRIG2.SLEVE, TRIG2.SWITCH; no longer TRIG1IN.SLEVE, TRIG1IN.SWITCH, TRIG2IN.SLEVE, TRIG2IN.SWITCH
- net N$1: now also TRIG2.TIP; no longer TRIG2IN.TIP
- net N$57: now also TRIG1.TIP; no longer TRIG1IN.TIP
Other:
- moved on the sheet: OUTA, OUTB
