File: peaks/hardware_design/pcb_banana/peaks_v02.brd (EAGLE design)
At the start: 38.7 x 106.7 mm, 94 parts, among them IC1 LM1117-3.3, IC2 LM4040B25, IC3 DAC8552, IC4 OPA2171, IC5 OPA2171, IC6 LM4040B10, Q1 8MHz, Q2 MMBT3904, Q3 MMBT3904

Commit message: adding rapid bananas
Parts:
- removed TRIG1IN, TRIG2IN: (no value), Jalco_3_5_jack:PJ-360_BANANA
- added TRIG1, TRIG2: WQP-PJ301BM, minijack_3_5_quingpu:WQP-PJ301BM
- OUTA, OUTB: value (none) -> WQP-PJ301BM; device Jalco_3_5_jack:PJ-360_BANANA -> minijack_3_5_quingpu:WQP-PJ301BM
- moved OUTA 0.64 mm to (21.0, 6.35), turned to 0 degrees
- moved OUTB 0.32 mm to (32.7, 6.35), turned to 0 degrees
- renumbered SWTRIG1 to SW6, SWTRIG2 to SW4
Connections:
- net GND: now also OUTA.G1, OUTA.G2, OUTB.G1, OUTB.G2, TRIG1.DESC, TRIG1.G1, TRIG1.G2, TRIG2.DESC, TRIG2.G1, TRIG2.G2; no longer OUTA.GND, OUTB.GND, TRIG1IN.6, TRIG1IN.GND, TRIG2IN.6, TRIG2IN.GND
- net N$1: now also TRIG2.TIP; no longer TRIG2IN.TIP
- net N$57: now also TRIG1.TIP; no longer TRIG1IN.TIP
Routing:
- net SW_TRIG_1: track 63.7 -> 58.6 mm, vias 1 -> 4
- net N$22: track 46.7 -> 42.8 mm, vias 2 -> 4
- net VEE: track 153.9 -> 156.3 mm, vias 3 -> 4
- net N$2: track 55.5 -> 57.5 mm
- net +3V3: track 167.0 -> 165.5 mm, vias 7 -> 11
- net TRIG_1: track 62.1 -> 63.4 mm
- net N$24: track 7.96 -> 9.28 mm
- net GND: vias 44 -> 42

Commit message: Fixes to peaks bananas
Routing:
- net GND: vias 42 -> 47
Changed lines of the file:
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@@
 <setting verticaltext="up"/>
 </settings>
-<grid distance="12.5" unitdist="mil" unit="mil" style="lines" multiple="4" display="yes" altdistance="0.025" altunitdist="inch" altunit="inch"/>
+<grid distance="0.000123" unitdist="mil" unit="mil" style="lines" multiple="4" display="yes" altdistance="0.025" altunitdist="inch" altunit="inch"/>
 <layers>
 <layer number="1" name="Top" color="4" fill="1" visible="yes" active="yes"/>
@@
 <wire x1="13.855" y1="73.1475" x2="13.855" y2="75.6801" width="0.254" layer="1"/>
 <via x="20.6375" y="46.6725" extent="1-16" drill="0.6"/>
-<via x="12.7" y="18.415" extent="1-16" drill="0.6"/>
-<via x="20.0025" y="29.845" extent="1-16" drill="0.6"/>
+<wire x1="21.9075" y1="20.955" x2="21.9075" y2="20.955" width="0" layer="19" extent="1-16"/>
+<via x="19.62715625" y="29.644778125" extent="1-16" drill="0.6"/>
 <via x="13.4938" y="76.0413" extent="1-16" drill="0.6"/>
 <via x="18.415" y="79.6925" extent="1-16" drill="0.6"/>
@@
 <via x="17.145" y="87.63" extent="1-16" drill="0.6"/>
 <via x="8.89" y="88.9" extent="1-16" drill="0.6"/>
-<via x="15.875" y="47.625" extent="1-16" drill="0.6"/>
+<via x="15.82495625" y="46.94925625" extent="1-16" drill="0.6"/>
 <via x="12.7" y="66.675" extent="1-16" drill="0.6"/>
-<via x="12.065" y="56.515" extent="1-16" drill="0.6"/>
+<via x="11.7475" y="56.515" extent="1-16" drill="0.6"/>
 <via x="24.765" y="27.94" extent="1-16" drill="0.6"/>
-<via x="16.51" y="26.67" extent="1-16" drill="0.6"/>
+<via x="16.409909375" y="26.644971875" extent="1-16" drill="0.6"/>
 <via x="24.765" y="33.3375" extent="1-16" drill="0.6"/>
 <via x="24.765" y="36.83" extent="1-16" drill="0.6"/>
@@
 <via x="10.4775" y="90.4875" extent="1-16" drill="0.6"/>
 <via x="23.495" y="60.6425" extent="1-16" drill="0.6"/>
-<via x="17.145" y="18.7325" extent="1-16" drill="0.6"/>
+<wire x1="23.1775" y1="18.0975" x2="23.1775" y2="18.0975" width="0" layer="19" extent="1-16"/>
 <via x="8.89" y="87.3125" extent="1-16" drill="0.6"/>
 <via x="8.89" y="85.725" extent="1-16" drill="0.6"/>
@@
 <contactref element="TRIG2" pad="G1"/>
 <wire x1="26.0375" y1="15.41" x2="24.17" y2="20.94" width="0" layer="19" extent="1-1"/>
+<via x="24.097178125" y="23.81105" extent="1-16" drill="0.6"/>
+<via x="8.255" y="20.6375" extent="1-16" drill="0.6"/>
+<via x="8.89" y="49.8475" extent="1-16" drill="0.6"/>
+<via x="34.29" y="35.56" extent="1-16" drill="0.6"/>
+<via x="26.9875" y="39.6875" extent="1-16" drill="0.6"/>
+<via x="16.940628125" y="18.355028125" extent="1-16" drill="0.6"/>
+<via x="17.4583125" y="38.481825" extent="1-16" drill="0.6"/>
 </signal>
 <signal name="+3V3">
